File: Hardware/SparkFun_IM19_IMU_Breakout.kicad_pcb (KiCad board)
At the start: 4 copper layers, 43.2 x 43.2 mm, 62 parts, among them J1 JST_Locking_4, J2 Conn_01x09, J3 USB_C_Receptacle, J4 Conn_01x09, U1 CH342F, U2 IM19, U3 74HC4066BQ, U4 RT9080-3.3

Commit message: More WIP
Parts:
- JP1: moved to B.Cu
- moved D3 24.9 mm to (152.1, 85.3), turned to 180 degrees
- moved D4 24.9 mm to (127.3, 85.3), turned to 0 degrees
- moved J2 20.3 mm to (149.9, 82.5), turned to 180 degrees
- moved C5 16.8 mm to (131.2, 116.2), turned to -90 degrees
- moved D2 8.14 mm to (118.2, 102.7)
- moved C8 7.27 mm to (125.7, 94.1)
- moved C9 7.21 mm to (125.7, 95.8)
- moved U4 7.18 mm to (125.7, 98.8)
- moved C11 7.15 mm to (125.7, 101.9)
- moved C12 7.10 mm to (125.7, 103.5)
- moved F1 5.08 mm to (119.4, 97.2)
- moved D1 3.97 mm to (120.5, 102.7)
- moved R3 2.54 mm to (151.1, 88.3)
- moved JP1 2.54 mm to (120.7, 92.7), turned to 0 degrees
- moved C3 2.45 mm to (130.4, 98.8), turned to -90 degrees
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Connections:
- D3 pad 1: TXD1 -> RXD2
- D3 pad 3: RXD2 -> TXD1
- D3 pad 4: TXD2 -> RXD1
- D3 pad 5: RXD1 -> TXD2
- D4 pad 1: TXD3 -> unconnected-(D4-K1-Pad1)
- D4 pad 3: unconnected-(D4-K2-Pad3) -> TXD3
- D4 pad 4: 3.3V -> RXD3
- D4 pad 5: RXD3 -> 3.3V
Routing:
- net BOOT: track 10.5 -> 11.5 mm
- net ~{RESET}: track 6.78 -> 7.45 mm
- net GND: vias 6 -> 38

Commit message: Add PWR LED and silk. Ignore -backups
Parts:
- removed kibuzzard-67DC4CF4: G***, kibuzzard-67DC4CF4
- removed kibuzzard-67DC4D0C: G***, kibuzzard-67DC4D0C
- removed the kibuzzard-67FFA928 at (176.3, 102.1)
- removed kibuzzard-6849609B: G***, kibuzzard-6849609B
- removed kibuzzard-68496623: G***, kibuzzard-68496623
- removed kibuzzard-68496634: G***, kibuzzard-68496634
- added D7: DF5A5.6LFU, SparkFun-Semiconductor-Standard:SOT-353, F.Cu at (151.9, 120.4)
- added G***: LOGO, SparkFun-Aesthetic:SparkFun_Logo_12.5mm, F.Cu at (149.1, 109.3)
- added G***: LOGO, SparkFun-Aesthetic:SparkFun_Logo_12.5mm, B.Cu at (137.2, 91.2)
- added PWR.1: ~, SparkFun-Jumper:Jumper_2_NC_Trace, B.Cu at (129.7, 105.7)
- added R6: 5.1k, SparkFun-Resistor:R_0603_1608Metric, F.Cu at (124.5, 107.3)
- added kibuzzard-68F5D5EE: G***, kibuzzard-68F5D5EE, F.Cu at (129.5, 120.8)
- added kibuzzard-68F5D5EE: G***, kibuzzard-68F5D5EE, B.Cu at (129.5, 120.8)
- added kibuzzard-68F5D651: G***, kibuzzard-68F5D651, F.Cu at (132.1, 120.9)
- added kibuzzard-68F5D651: G***, kibuzzard-68F5D651, B.Cu at (132.1, 120.9)
- added kibuzzard-68F5D664: G***, kibuzzard-68F5D664, F.Cu at (134.6, 120.8)
- added kibuzzard-68F5D664: G***, kibuzzard-68F5D664, B.Cu at (134.6, 120.8)
- added kibuzzard-68F5D677: G***, kibuzzard-68F5D677, F.Cu at (137.2, 119.0)
- added kibuzzard-68F5D677: G***, kibuzzard-68F5D677, B.Cu at (137.2, 119.0)
- added kibuzzard-68F5D6B2: G***, kibuzzard-68F5D6B2, F.Cu at (139.7, 120.4)
- added kibuzzard-68F5D6B2: G***, kibuzzard-68F5D6B2, B.Cu at (139.7, 120.4)
- added kibuzzard-68F5D6C3: G***, kibuzzard-68F5D6C3, F.Cu at (142.2, 120.1)
- added kibuzzard-68F5D6C3: G***, kibuzzard-68F5D6C3, B.Cu at (142.2, 120.1)
- added kibuzzard-68F5D6DA: G***, kibuzzard-68F5D6DA, F.Cu at (144.8, 120.8)
- added kibuzzard-68F5D6DA: G***, kibuzzard-68F5D6DA, B.Cu at (144.8, 120.8)
- added kibuzzard-68F5D706: G***, kibuzzard-68F5D706, F.Cu at (147.3, 120.8)
- added kibuzzard-68F5D706: G***, kibuzzard-68F5D706, B.Cu at (147.3, 120.8)
- added kibuzzard-68F5D71D: G***, kibuzzard-68F5D71D, F.Cu at (149.9, 119.8)
- added kibuzzard-68F5D71D: G***, kibuzzard-68F5D71D, B.Cu at (149.9, 119.7)
- added kibuzzard-68F5D97A: G***, kibuzzard-68F5D97A, F.Cu at (151.1, 89.5)
- added kibuzzard-68F5D9B9: G***, kibuzzard-68F5D9B9, F.Cu at (151.0, 92.1)
- added kibuzzard-68F5D9CC: G***, kibuzzard-68F5D9CC, F.Cu at (151.1, 90.8)
- added kibuzzard-68F5D9E8: G***, kibuzzard-68F5D9E8, F.Cu at (151.2, 93.3)
- added kibuzzard-68F5DA6F: G***, kibuzzard-68F5DA6F, F.Cu at (129.5, 85.0)
- added kibuzzard-68F5DA6F: G***, kibuzzard-68F5DA6F, B.Cu at (129.5, 85.0)
- added kibuzzard-68F5DABB: G***, kibuzzard-68F5DABB, F.Cu at (132.1, 84.4)
- added kibuzzard-68F5DABB: G***, kibuzzard-68F5DABB, B.Cu at (132.1, 84.4)
- added kibuzzard-68F5DAD8: G***, kibuzzard-68F5DAD8, F.Cu at (134.6, 84.8)
- added kibuzzard-68F5DAD8: G***, kibuzzard-68F5DAD8, B.Cu at (134.6, 84.8)
- added kibuzzard-68F5DB0E: G***, kibuzzard-68F5DB0E, F.Cu at (137.2, 85.1)
- added kibuzzard-68F5DB0E: G***, kibuzzard-68F5DB0E, B.Cu at (137.2, 85.1)
- added kibuzzard-68F5DB1B: G***, kibuzzard-68F5DB1B, F.Cu at (139.7, 85.1)
- added kibuzzard-68F5DB2C: G***, kibuzzard-68F5DB2C, F.Cu at (142.2, 85.1)
- added kibuzzard-68F5DB2C: G***, kibuzzard-68F5DB2C, B.Cu at (142.2, 85.1)
- added kibuzzard-68F5DB3E: G***, kibuzzard-68F5DB3E, F.Cu at (144.8, 85.1)
- added kibuzzard-68F5DB3E: G***, kibuzzard-68F5DB3E, B.Cu at (144.8, 85.1)
- added kibuzzard-68F5DB51: G***, kibuzzard-68F5DB51, F.Cu at (147.3, 85.0)
- added kibuzzard-68F5DB51: G***, kibuzzard-68F5DB51, B.Cu at (147.3, 85.0)
- added kibuzzard-68F5DB62: G***, kibuzzard-68F5DB62, F.Cu at (149.9, 85.0)
- added kibuzzard-68F5DB62: G***, kibuzzard-68F5DB62, B.Cu at (149.9, 85.0)
- added kibuzzard-68F5DDAB: G***, kibuzzard-68F5DDAB, B.Cu at (117.2, 111.8)
- added kibuzzard-68F5DDD0: G***, kibuzzard-68F5DDD0, B.Cu at (125.7, 109.0)
- added kibuzzard-68F5DDF5: G***, kibuzzard-68F5DDF5, B.Cu at (125.7, 114.4)
- added kibuzzard-68F5DE2E: G***, kibuzzard-68F5DE2E, B.Cu at (136.8, 111.8)
- added kibuzzard-68F5E094: G***, kibuzzard-68F5E094, F.Cu at (149.1, 112.4)
- added kibuzzard-68F5E094: G***, kibuzzard-68F5E094, B.Cu at (137.2, 94.2)
- added kibuzzard-68F5E0B5: G***, kibuzzard-68F5E0B5, F.Cu at (149.2, 114.9)
- added kibuzzard-68F5E0B5: G***, kibuzzard-68F5E0B5, B.Cu at (137.1, 96.8)
- added kibuzzard-68F5E8F0: G***, kibuzzard-68F5E8F0, B.Cu at (139.7, 85.1)
- added kibuzzard-68F5E8FA: G***, kibuzzard-68F5E8FA, F.Cu at (129.7, 108.5)
- added kibuzzard-68F5E982: G***, kibuzzard-68F5E982, B.Cu at (126.6, 105.7)
- added kibuzzard-68F5E9AB: G***, kibuzzard-68F5E9AB, B.Cu at (153.4, 91.2)
- added kibuzzard-68F5E9C6: G***, kibuzzard-68F5E9C6, B.Cu at (156.2, 88.8)
- added kibuzzard-68F5E9E3: G***, kibuzzard-68F5E9E3, B.Cu at (156.2, 93.7)
- added kibuzzard-68F5EA91: G***, kibuzzard-68F5EA91, F.Cu at (120.7, 90.8)
- added kibuzzard-68F5EA91: G***, kibuzzard-68F5EA91, B.Cu at (120.7, 90.8)
- added kibuzzard-68F5EC7C: G***, kibuzzard-68F5EC7C, B.Cu at (137.5, 104.4)
- added kibuzzard-68F5ECB4: G***, kibuzzard-68F5ECB4, B.Cu at (137.5, 105.7)
- added kibuzzard-68F5ECF3: G***, kibuzzard-68F5ECF3, B.Cu at (137.5, 106.8)
- added kibuzzard-68F5EDC8: G***, kibuzzard-68F5EDC8, B.Cu at (137.5, 107.9)
- C10: value 10uF -> 1.0uF
- C11: value 1.0uF -> 10uF
- D3: value DF5A5.6LFU -> Red; footprint SparkFun-Semiconductor-Standard:SOT-353 -> SparkFun-LED:LED_0603_1608Metric_Red
- D5: value DT1042-04SO -> DF5A5.6LFU; footprint SparkFun-Semiconductor-Standard:SOT23-6 -> SparkFun-Semiconductor-Standard:SOT-353
- D6: value DF5A5.6LFU -> DT1042-04SO; footprint SparkFun-Semiconductor-Standard:SOT-353 -> SparkFun-Semiconductor-Standard:SOT23-6
- R4: value 5.1k -> 4.7k
- U3: value 74HC4066BQ -> RT9080-3.3; footprint SparkFun-Semiconductor-Standard:QFN-14_2.5x3mm_P0.5mm_EP1x1.5mm -> SparkFun-Semiconductor-Standard:SOT23-5
- U4: value RT9080-3.3 -> 74HC4066BQ; footprint SparkFun-Semiconductor-Standard:SOT23-5 -> SparkFun-Semiconductor-Standard:QFN-14_2.5x3mm_P0.5mm_EP1x1.5mm
- kibuzzard-67FFA928, kibuzzard-67FFB450, kibuzzard-67FFB45E, kibuzzard-67FFB46A: moved to F.Cu
- kibuzzard-67FFB450, kibuzzard-67FFB45E, kibuzzard-67FFB46A: moved to B.Cu
- moved kibuzzard-67FFB45E 40.8 mm to (137.2, 99.8), turned to 0 degrees
- moved kibuzzard-67FFB46A 37.5 mm to (136.1, 102.9), turned to 180 degrees
- moved kibuzzard-67FFB450 34.4 mm to (140.5, 102.9), turned to 180 degrees
- moved D3 31.4 mm to (129.7, 107.3)
- moved D6 27.8 mm to (125.7, 111.8), turned to 0 degrees
- moved Ref** 26.6 mm to (123.8, 120.6)
- moved D5 26.5 mm to (127.5, 85.3)
- moved C10 26.4 mm to (125.7, 101.9)
- moved C11 26.4 mm to (151.1, 94.6)
- moved D4 24.6 mm to (151.9, 85.3), turned to 180 degrees
- moved R1 24.5 mm to (121.9, 97.2), turned to 90 degrees
- moved R2 24.5 mm to (141.6, 111.8), turned to 0 degrees
- moved kibuzzard-67FFB46A 24.0 mm to (150.3, 102.9), turned to 0 degrees
- moved kibuzzard-67FFB45E 23.7 mm to (151.3, 99.8), turned to 0 degrees
- moved kibuzzard-67FFA928 23.5 mm to (153.2, 101.6), turned to 0 degrees
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Connections:
- C10 pad 1: Net-(J1-Pin_1) -> 3.3V
- C11 pad 1: 3.3V -> Net-(J1-Pin_1)
- D3 pad 1: RXD2 -> GND
- D3 pad 2: GND -> Net-(D3-A)
- D4 pad 1: unconnected-(D4-K1-Pad1) -> RXD2
- D4 pad 3: TXD3 -> TXD1
- D4 pad 4: RXD3 -> RXD1
- D4 pad 5: 3.3V -> TXD2
- D5 pad 1: D+ -> unconnected-(D5-K1-Pad1)
- D5 pad 3: D- -> TXD3
- D5 pad 4: D- -> RXD3
- D5 pad 5: VUSB -> 3.3V
- D6 pad 1: ~{RESET} -> D+
- D6 pad 3: GPIO -> D-
- D6 pad 4: BOOT -> D-
- D6 pad 5: PPS -> VUSB
- R1 pad 1: CH342_EN -> 3V3_EN
- R1 pad 2: 3.3V -> 5V
- R2 pad 1: 3V3_EN -> CH342_EN
- R2 pad 2: 5V -> 3.3V
- R4 pad 1: GND -> Net-(D3-A)
- R4 pad 2: Net-(J3-CC2) -> Net-(PWR.1-A)
- R5 pad 2: Net-(J3-CC1) -> Net-(J3-CC2)
- U3 pad 1: Net-(U1-TXD0) -> 5V
- U3 pad 2: RXD1 -> GND
- U3 pad 3: TXD1 -> 3V3_EN
- U3 pad 4: Net-(U1-RXD0) -> unconnected-(U3-NC-Pad4)
- U3 pad 5: CH342_EN -> 3.3V
- U4 pad 1: 5V -> Net-(U1-TXD0)
- U4 pad 2: GND -> RXD1
- U4 pad 3: 3V3_EN -> TXD1
- U4 pad 4: unconnected-(U4-NC-Pad4) -> Net-(U1-RXD0)
- U4 pad 5: 3.3V -> CH342_EN

Commit message: Routed
Parts:
- added TP3: 1.25mm, SparkFun-Connector:TestPoint-1.25mm, B.Cu at (128.1, 111.8)
- added kibuzzard-68F62121: G***, kibuzzard-68F62121, B.Cu at (129.4, 111.8)
- moved SHLD1 1.78 mm to (117.1, 111.8)
- moved kibuzzard-68F5DDAB 1.65 mm to (118.9, 111.8)
- moved R5 0.51 mm to (125.0, 116.2)
- moved R6 0.51 mm to (125.0, 107.3)
- moved kibuzzard-68F5DDD0 0.13 mm to (125.7, 109.1)
Routing:
- net 5V: track 0.00 -> 62.3 mm, vias 0 -> 4
- net 3V3_EN: track 0.00 -> 54.5 mm, vias 0 -> 3
- net TXD1: track 4.14 -> 53.2 mm, vias 0 -> 3
- net ~{RESET}: track 7.20 -> 54.1 mm, vias 0 -> 3
- net RXD1: track 4.66 -> 49.6 mm, vias 0 -> 3
- net BOOT: track 11.2 -> 54.2 mm, vias 0 -> 3
- net TXD2: track 7.74 -> 49.7 mm, vias 0 -> 2
- net RXD2: track 13.1 -> 52.3 mm, vias 0 -> 2
- net RXD3: track 10.3 -> 48.7 mm, vias 0 -> 3
- net TXD3: track 15.6 -> 53.9 mm, vias 0 -> 3
- net 3.3V: track 7.20 -> 44.6 mm, vias 0 -> 11
- net GPIO: track 15.3 -> 50.3 mm, vias 0 -> 2
- net VUSB: track 0.00 -> 33.4 mm, vias 0 -> 4
- net VIN: track 0.00 -> 32.9 mm, vias 0 -> 2
- net PPS: track 7.20 -> 35.5 mm, vias 0 -> 2
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